File: Andromeda.kicad_sch (KiCad schematic)
At the start: 30 parts, among them J1 Barrel_Jack, J2 USB_C_Receptacle_USB2.0, M1 Motor_DC, SW1 Reset, SW2 Boot, SW4 SW_DIP_x01, U1 ESP32-S2-SOLO, U2 DRV8871DDA, U3 AP2127K-3.3

Commit message: Complete rough schematic
Parts:
- removed D2: LED, Diode_SMD:D_1206_3216Metric, symbol Device:LED
- removed M1: Motor_DC, Connector_Wire:SolderWire-0.75sqmm_1x02_P7mm_D1.25mm_OD3.5mm, symbol Motor:Motor_DC
- removed R4: 30k, Resistor_SMD:R_0805_2012Metric, symbol Device:R
- removed SW4: SW_DIP_x01, Connector_Wire:SolderWire-2.5sqmm_1x02_P7.2mm_D2.4mm_OD3.6mm, symbol Switch:SW_DIP_x01
- removed U2: DRV8871DDA, Package_SO:Texas_HTSOP-8-1EP_3.9x4.9mm_P1.27mm_EP2.95x4.9mm_Mask2.4x3.1mm_ThermalVias, symbol Driver_Motor:DRV8871DDA
- added C10, C12, C15, C16, C18, C20, C21, C22, C23, C24, C7, C8, C9: 0.1uF, symbol Device:C_Small
- added C11: 10uF, symbol Device:C_Small
- added C13, C14: 22uF, symbol Device:C_Small
- added F2: Fuse_Small, Fuse:Fuse_0805_2012Metric, symbol Device:Fuse_Small
- added J10, J3, J4, J5, J6, J7, J8, J9: RJ45, symbol Connector:RJ45
- added J11: Conn_02x08_Counter_Clockwise_MountingPin, symbol Connector_Generic_MountingPin:Conn_02x08_Counter_Clockwise_MountingPin
- added L1: 4.7uH, symbol Device:L_Small
- added R10, R11, R14, R15, R16, R17, R18, R19, R20, R21, R4, R5, R6, R7, R8: 1K, symbol Device:R_Small
- added U10, U4, U9: TXB0108DQSR, Package_SON:USON-20_2x4mm_P0.4mm, symbol Logic_LevelTranslator:TXB0108DQSR
- added U2, U6, U7, U8: DRV8212DSGR, WSON_212DSGR_TEX, symbol DRV8870DDA:DRV8212DSGR
- added U5: AP63205WU, Package_TO_SOT_SMD:TSOT-23-6, symbol Regulator_Switching:AP63205WU
- C17: footprint Capacitor_SMD:C_0805_2012Metric -> (none)
- C19: value 47uF -> 0.1uF; footprint Capacitor_SMD:C_0805_2012Metric -> (none)
- F1: footprint (none) -> Fuse:Fuse_0805_2012Metric
- R3: value 150 -> 1K; footprint Resistor_SMD:R_0603_1608Metric -> (none)
Connections:
- net +3.3V: now also C10.2, C16.1, C18.1, C20.1, C21.2, C23.2, C7.1, J10.3, J7.3, J8.3, J9.3, R20.1, R21.1, R6.1, U10.5 (VCCA), U2.8 (VCC), U4.5 (VCCA), U6.8 (VCC), U7.8 (VCC), U8.8 (VCC), U9.5 (VCCA)
- net +5V: now also C1.1, U3.1 (VIN), C13.1, C14.1, C22.2, C24.2, C9.2, F2.2, J10.5, J3.5, J4.5, J5.5, J6.5, J7.5, J8.5, J9.5, L1.2, U10.16 (VCCB), U4.16 (VCCB), U5.1 (FB), U9.16 (VCCB); no longer D4.1 (K), R3.1
- net GND: now also R3.2, C10.1, C11.2, C13.2, C14.2, C15.2, C16.2, C18.2, C20.2, C21.1, C22.1, C23.1, C24.1, C7.2, C8.2, C9.1, J10.6, J11.1 (Pin_1), J11.2 (Pin_2), J11.3 (Pin_3), J11.4 (Pin_4), J11.5 (Pin_5), J11.6 (Pin_6), J11.7 (Pin_7), J11.8 (Pin_8), J3.6, J4.6, J5.6, J6.6, J7.6, J8.6, J9.6, R10.2, R11.2, R14.2, R15.2, R16.2, R17.2, R18.2, R19.2, R4.2, R5.2, R8.2, U10.15 (GND), U2.4 (GND), U4.15 (GND), U5.4 (GND), U6.4 (GND), U7.4 (GND), U8.4 (GND), U9.15 (GND)
- net GPIO10: now also U10.2 (A2)
- net GPIO11: now also U10.3 (A3)
- net GPIO12: now also U10.4 (A4)
- net GPIO13: now also U10.7 (A5)
- net GPIO21: now also U4.3 (A3)
- net GPIO33: now also U4.4 (A4)
- net GPIO34: now also U4.7 (A5)
- net GPIO35: now also U4.8 (A6)
- net GPIO36: now also U4.9 (A7)
- net GPIO4: now also U9.4 (A4)
- net GPIO9: now also U10.1 (A1)
- net GPIO17: now reaches U1.10 (GPIO17/U1TXD/ADC2_CH6/DAC_1)
- net GPIO17: now also U4.1 (A1)
- net GPIO18: now reaches U1.11 (GPIO18/U1RXD/ADC2_CH7/DAC_2/CLK_OUT3)
- net GPIO18: now also U4.2 (A2)
- net GPIO8: now reaches U1.12 (GPIO8/TOUCH8/ADC1_CH7)
- net GPIO8: now also U9.10 (A8)
- net GPIO3: now reaches U1.15 (GPIO3/TOUCH3/ADC1_CH2)
- net GPIO3: now also U9.3 (A3)
- net GPIO14: now reaches U1.22 (GPIO14/TOUCH14/ADC2_CH3/FSPIWP/FSPIDQS)
- net GPIO14: now also U10.8 (A6)
- net GPIO45: now reaches U1.26 (GPIO45)
- net GPIO45: now also U4.10 (A8)
- net GPIO37: now reaches U1.30 (SPIDQS/GPIO37/FSPIQ)
- net GPIO37: now also U7.6 (IN1/PH)
- net GPIO38: now reaches U1.31 (GPIO38/FSPIWP)
- net GPIO38: now also R3.1, U7.5 (IN2/EN)
- net GPIO39: now reaches U1.32 (MTCK/GPIO39/CLK_OUT3)
- net GPIO39: now also U2.6 (IN1/PH)
- net GPIO40: now reaches U1.33 (MTDO/GPIO40/CLK_OUT2)
- net GPIO40: now also R8.1, U2.5 (IN2/EN)
- net GPIO41: now reaches U1.34 (MTDI/GPIO41/CLK_OUT1)
- net GPIO41: now also U6.6 (IN1/PH)
- net GPIO42: now reaches U1.35 (MTMS/GPIO42)
- net GPIO42: now also R14.1, U6.5 (IN2/EN)
- net GPIO44: now reaches U1.36 (U0RXD/GPIO44/CLK_OUT2)
- net GPIO44: now also R17.1, U8.5 (IN2/EN)
- net GPIO43: now reaches U1.37 (U0TXD/GPIO43/CLK_OUT1)
- net GPIO43: now also U8.6 (IN1/PH)
- net GPIO2: now reaches U1.38 (GPIO2/TOUCH2/ADC1_CH1)
- net GPIO2: now also U9.2 (A2)
- net GPIO1: now reaches U1.39 (GPIO1/TOUCH1/ADC1_CH0)
- net GPIO1: now also U9.1 (A1)
- net GPIO5: now reaches U1.5 (GPIO5/TOUCH5/ADC1_CH4)
- net GPIO5: now also U9.7 (A5)
- net GPIO6: now reaches U1.6 (GPIO6/TOUCH6/ADC1_CH5)
- net GPIO6: now also U9.8 (A6)
- net GPIO7: now reaches U1.7 (GPIO7/TOUCH7/ADC1_CH6)
- net GPIO7: now also U9.9 (A7)
- net GPIO15: now reaches U1.8 (GPIO15/U0RTS/ADC2_CH4/XTAL_32K_P)
- net GPIO15: now also U10.9 (A7)
- net GPIO16: now reaches U1.9 (GPIO16/U0CTS/ADC2_CH5/XTAL_32K_N)
- net GPIO16: now also U10.10 (A8)
- net +12V renamed +VBATT
- net +VBATT: now also F1.2, TP3.1, C11.1, C15.1, C8.1, J3.4, J4.4, J5.4, J6.4, R7.1, U2.1 (VM), U5.3 (IN), U6.1 (VM), U7.1 (VM), U8.1 (VM)
- removed net +6V: C1.1, F1.2, TP3.1, U3.1 (VIN)
- new net: R21.2, U10.6 (OE)
- new net: J4.2, U2.2 (OUT1)
- new net: J4.1, U2.3 (OUT2)
- new net: R10.1, R11.1, U2.7 (MODE)
- new net: R6.2, U4.6 (OE)
- new net: J6.2, U8.2 (OUT1)
- new net: J6.1, U8.3 (OUT2)
- new net: R18.1, R19.1, U8.7 (MODE)
- new net: R4.1, R5.1, U7.7 (MODE)
- new net: J5.1, U6.3 (OUT2)
- new net: J5.2, U6.2 (OUT1)
- new net: J3.2, U7.2 (OUT1)
- new net: J3.1, U7.3 (OUT2)
- new net: D4.1 (K), F2.1
- new net: R15.1, R16.1, U6.7 (MODE)
- new net: R7.2, U5.2 (EN)
- new net: C12.2, U5.5 (SW)
- new net: C12.1, L1.1, U5.6 (BST)
- new net: R20.2, U9.6 (OE)
- new net BREAKOUT_1: J11.16 (Pin_16), U10.20 (B1)
- new net BREAKOUT_2: J11.15 (Pin_15), U10.19 (B2)
- new net BREAKOUT_3: J11.14 (Pin_14), U10.18 (B3)
- new net BREAKOUT_4: J11.13 (Pin_13), U10.17 (B4)
- new net BREAKOUT_5: J11.12 (Pin_12), U10.14 (B5)
- new net BREAKOUT_6: J11.11 (Pin_11), U10.13 (B6)
- new net BREAKOUT_7: J11.10 (Pin_10), U10.12 (B7)
- new net BREAKOUT_8: J11.9 (Pin_9), U10.11 (B8)
- new net ENC1A: J3.7, U4.20 (B1)
- new net ENC1B: J3.8, U4.19 (B2)
- new net ENC2A: J4.7, U4.18 (B3)
- new net ENC2B: J4.8, U4.17 (B4)
- new net ENC3A: J5.7, U4.14 (B5)
- new net ENC3B: J5.8, U4.13 (B6)
- new net ENC4A: J6.7, U4.12 (B7)
- new net ENC4B: J6.8, U4.11 (B8)
- new net SIG_INPUT_1: J7.7, U9.20 (B1)
- new net SIG_INPUT_2: J7.8, U9.19 (B2)
- new net SIG_INPUT_3: J8.7, U9.18 (B3)
- new net SIG_INPUT_4: J8.8, U9.17 (B4)
- new net SIG_INPUT_5: J9.7, U9.14 (B5)
- new net SIG_INPUT_6: J9.8, U9.13 (B6)
- new net SIG_INPUT_7: J10.7, U9.12 (B7)
- new net SIG_INPUT_8: J10.8, U9.11 (B8)
- no-connect marks 24 -> 20
Other:
- note added: "5V Supply"
- note added: "Breakout"
- note added: "Logic Shifter"
- note added: "Sensor Input"
- moved on the sheet: C1, C2, C3, C4, C5, C6, D3, D4, F1, J1, J2, R1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

Commit message: Pass ERC
Parts:
- added SW3: SW_Nidec_CAS-120A1, Button_Switch_SMD:Nidec_Copal_CAS-120A, symbol Switch:SW_Nidec_CAS-120A1
- J1: footprint Connector_BarrelJack:BarrelJack_CUI_PJ-036AH-SMT_Horizontal -> CUI_PJ-036AH-SMT-TR
- J2: symbol Connector:USB_C_Receptacle_USB2.0 -> Connector:USB_C_Receptacle_USB2.0_16P
- U1: symbol esp32:ESP32-S2-SOLO -> PCM_Espressif:ESP32-S2-SOLO
Connections:
- net +5V: no longer C1.1, U3.1 (VIN)
- net at F1.1: now also SW3.1 (C); no longer J1.1
- net +VBATT renamed +6V
- net +6V: now also C1.1, U3.1 (VIN)
- new net: J1.1, SW3.2 (B)
- no-connect marks 20 -> 21
Other:
- note added: "6V Supply"
- note removed: "5V Supply"
- moved on the sheet: C10, C21, C22, C23, C24, C3, C4, C5, C6, C9, F1, J1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

Commit message: Remove Logic Level Shifters
Parts:
- removed C10, C21, C22, C23, C24, C9: 0.1uF, symbol Device:C_Small
- removed R20, R21, R6: 1K, symbol Device:R_Small
- removed U10, U4, U9: TXB0108DQSR, Package_SON:USON-20_2x4mm_P0.4mm, symbol Logic_LevelTranslator:TXB0108DQSR
Connections:
- net BREAKOUT_1 is gone; now on net GPIO9: J11.16 (Pin_16)
- net BREAKOUT_2 is gone; now on net GPIO10: J11.15 (Pin_15)
- net BREAKOUT_3 is gone; now on net GPIO11: J11.14 (Pin_14)
- net BREAKOUT_4 is gone; now on net GPIO12: J11.13 (Pin_13)
- net BREAKOUT_5 is gone; now on net GPIO13: J11.12 (Pin_12)
- net BREAKOUT_6 is gone; now on net GPIO14: J11.11 (Pin_11)
- net BREAKOUT_7 is gone; now on net GPIO15: J11.10 (Pin_10)
- net BREAKOUT_8 is gone; now on net GPIO16: J11.9 (Pin_9)
- net ENC1A is gone; now on net GPIO17: J3.7
- net ENC1B is gone; now on net GPIO18: J3.8
- net ENC2A is gone; now on net GPIO21: J4.7
- net ENC2B is gone; now on net GPIO33: J4.8
- net ENC3A is gone; now on net GPIO34: J5.7
- net ENC3B is gone; now on net GPIO35: J5.8
- net ENC4A is gone; now on net GPIO36: J6.7
- net ENC4B is gone; now on net GPIO45: J6.8
- net SIG_INPUT_1 is gone; now on net GPIO1: J7.7
- net SIG_INPUT_2 is gone; now on net GPIO2: J7.8
- net SIG_INPUT_3 is gone; now on net GPIO3: J8.7
- net SIG_INPUT_4 is gone; now on net GPIO4: J8.8
- net SIG_INPUT_5 is gone; now on net GPIO5: J9.7
- net SIG_INPUT_6 is gone; now on net GPIO6: J9.8
- net SIG_INPUT_7 is gone; now on net GPIO7: J10.7
- net SIG_INPUT_8 is gone; now on net GPIO8: J10.8
- net +3.3V: now also J3.5, J4.5, J5.5, J6.5
- net +5V: no longer J3.5, J4.5, J5.5, J6.5
Other:
- note added: "5V Supply"
- note removed: "6V Supply"
- note removed: "Logic Shifter"
- moved on the sheet: J11

Commit message: Fix  some weirdness
Parts:
- removed C19, C20: 0.1uF, symbol Device:C_Small
- removed J11: Conn_02x08_Counter_Clockwise_MountingPin, symbol Connector_Generic_MountingPin:Conn_02x08_Counter_Clockwise_MountingPin
- removed U8: DRV8212DSGR, WSON_212DSGR_TEX, symbol DRV8870DDA:DRV8212DSGR
- added C10, C9: 0.1uF, symbol Device:C_Small
- added J11: Conn_01x08_Pin, symbol Connector:Conn_01x08_Pin
- added J12, J13: RJ45, symbol Connector:RJ45
- added R20, R21, R22, R23, R24, R25, R26, R27, R28, R29, R30, R31, R32, R33, R34, R6: 1K, symbol Device:R_Small
- added U4: DRV8212DSGR, WSON_212DSGR_TEX, symbol DRV8870DDA:DRV8212DSGR
Connections:
- net +3.3V: now also C17.1, J10.5, J7.5, J8.5, J9.5, C10.1, J11.5 (Pin_5), J11.6 (Pin_6), J12.5, J13.5, U4.8 (VCC); no longer C7.1, J10.3, J7.3, J8.3, J9.3
- net +5V: now also J11.7 (Pin_7); no longer J10.5, J7.5, J8.5, J9.5
- net +6V: now also C7.1, C9.1, U4.1 (VM); no longer C17.1
- net GND: now also C10.2, C9.2, J11.8 (Pin_8), J12.6, J13.6, R6.2, U4.4 (GND); no longer R10.2, R14.2, R15.2, R16.2, R17.2, R18.2, R19.2, R5.2, R8.2
- net GPIO1: now also R19.2; no longer J7.7
- net GPIO10: now also R28.2
- net GPIO11: now also R29.2
- net GPIO12: now also R30.2
- net GPIO13: now also R31.1
- net GPIO14: now also R32.1
- net GPIO15: now also R33.1
- net GPIO16: now also R34.1
- net GPIO17: now also R5.2; no longer J3.7
- net GPIO18: now also R8.2; no longer J3.8
- net GPIO2: now also R20.2; no longer J7.8
- net GPIO21: now also R17.2; no longer J4.7
- net GPIO3: now also R21.2; no longer J8.7
- net GPIO33: now also R18.2; no longer J4.8
- net GPIO34: now also R10.2; no longer J5.7
- net GPIO35: now also R14.2; no longer J5.8
- net GPIO36: now also R15.2; no longer J6.7
- net GPIO37: now also U6.6 (IN1/PH); no longer U7.6 (IN1/PH)
- net GPIO38: now also U6.5 (IN2/EN); no longer R3.1, U7.5 (IN2/EN)
- net GPIO4: now also R22.2; no longer J8.8
- net GPIO40: no longer R8.1
- net GPIO41: now also U7.6 (IN1/PH); no longer U6.6 (IN1/PH)
- net GPIO42: now also U7.5 (IN2/EN); no longer R14.1, U6.5 (IN2/EN)
- net GPIO43: now also U4.6 (IN1/PH)
- net GPIO44: now also U4.5 (IN2/EN); no longer R17.1
- net GPIO45: now also R16.2; no longer J6.8
- net GPIO5: now also R23.2; no longer J9.7
- net GPIO6: now also R24.2; no longer J9.8
- net GPIO7: now also R25.2; no longer J10.7
- net GPIO8: now also R26.2; no longer J10.8
- net GPIO9: now also R27.2
- net at R11.1, U2.7 (MODE): no longer R10.1
- net at J6.2: now also U4.2 (OUT1)
- net at J6.1: now also U4.3 (OUT2)
- net at R18.1: now also J4.8; no longer R19.1
- net at R4.1, U7.7 (MODE): no longer R5.1
- net at U6.3 (OUT2): now also J3.1; no longer J5.1
- net at U6.2 (OUT1): now also J3.2; no longer J5.2
- net at U7.2 (OUT1): now also J5.2; no longer J3.2
- net at U7.3 (OUT2): now also J5.1; no longer J3.1
- new net: J5.8, R14.1
- new net: J13.8, R30.1
- new net: J13.7, R29.1
- new net: J6.7, R15.1
- new net: J6.8, R16.1
- new net: J11.1 (Pin_1), R31.2
- new net: J4.7, R17.1
- new net: J11.4 (Pin_4), R34.2
- new net: J7.7, R19.1
- new net: J7.8, R20.1
- new net: J11.2 (Pin_2), R32.2
- new net: J11.3 (Pin_3), R33.2
- new net: J12.7, R27.1
- new net: J9.7, R23.1
- new net: R3.1, U6.7 (MODE)
- new net: J8.7, R21.1
- new net: J8.8, R22.1
- new net: J10.8, R26.1
- new net: J10.7, R25.1
- new net: J9.8, R24.1
- new net: J12.8, R28.1
- new net: J3.8, R8.1
- new net: J5.7, R10.1
- new net: J3.7, R5.1
- new net: R6.1, U4.7 (MODE)
- no-connect marks 21 -> 32
Other:
- moved on the sheet: C15, C16, J4, R11

Commit message: begin layout
Parts:
- C10, C11, C12, C13, C14, C15, C16, C17, C18, C7, C8, C9: footprint (none) -> Capacitor_SMD:C_0805_2012Metric
- C2, C5: footprint Capacitor_SMD:C_0603_1608Metric -> Capacitor_SMD:C_0805_2012Metric
- J1: footprint CUI_PJ-036AH-SMT-TR -> Connector_BarrelJack:BarrelJack_CUI_PJ-036AH-SMT_Horizontal
- J10, J12, J13, J3, J4, J5, J6, J7, J8, J9: footprint (none) -> Connector_RJ:RJ45_Amphenol_54602-x08_Horizontal
- J11: footprint (none) -> Connector_PinHeader_2.54mm:PinHeader_2x08_P2.54mm_Vertical
- L1: footprint (none) -> Inductor_THT:L_Radial_D9.5mm_P5.00mm_Fastron_07HVP
- R10, R11, R14, R15, R16, R17, R18, R19, R20, R21, R22, R23, R24, R25, R26, R27, R28, R29, R3, R30, R31, R32, R33, R34, R4, R5, R6, R7, R8: footprint (none) -> Resistor_SMD:R_0805_2012Metric
- R9: footprint Resistor_SMD:R_0603_1608Metric -> Resistor_SMD:R_0805_2012Metric
- U2, U4, U6, U7: footprint WSON_212DSGR_TEX -> DRV8870DDA:WSON_212DSGR_TEX
Connections:
- net at U2.2 (OUT1): now also J4.1; no longer J4.2
- net at U2.3 (OUT2): now also J4.2; no longer J4.1
- net at J6.1: now also U4.2 (OUT1); no longer U4.3 (OUT2)
- net at J6.2: now also U4.3 (OUT2); no longer U4.2 (OUT1)
- net at U6.2 (OUT1): now also J3.1; no longer J3.2
- net at U6.3 (OUT2): now also J3.2; no longer J3.1
- net at U7.2 (OUT1): now also J5.1; no longer J5.2
- net at U7.3 (OUT2): now also J5.2; no longer J5.1

Commit message: Switch to 5V, Add Gyro, GPIO extender
Parts:
- removed R19, R20, R5: 1K, Resistor_SMD:R_0805_2012Metric, symbol Device:R_Small
- removed U1: ESP32-S2-SOLO, PCM_Espressif:ESP32-S2-SOLO, symbol PCM_Espressif:ESP32-S2-SOLO
- added C19, C20, C21, C23: .1uF, Capacitor_SMD:C_0805_2012Metric, symbol Device:C
- added C22: 10nF, Capacitor_SMD:C_0805_2012Metric, symbol Device:C_Small
- added C24: 0.1uF, Capacitor_SMD:C_0805_2012Metric, symbol Device:C_Small
- added C25: 2.2uF, Capacitor_SMD:C_0805_2012Metric, symbol Device:C_Small
- added MT1: ICM-42670-P, ICM-42670-P:XDCR_ICM-42670-P, symbol ICM-42670-P:ICM-42670-P
- added R13, R40, R41, R48, R50, R7, R9: 1K, Resistor_SMD:R_0805_2012Metric, symbol Device:R_Small
- added R35, R43, R52: 20K, Resistor_SMD:R_0805_2012Metric, symbol Device:R_Small
- added R36, R37, R38, R39, R42, R44, R45, R46, R47, R49, R51: 10K, Resistor_SMD:R_0805_2012Metric, symbol Device:R_Small
- added U5: ESP32-S3-WROOM-1, PCM_Espressif:ESP32-S3-WROOM-1, symbol PCM_Espressif:ESP32-S3-WROOM-1
- added U8: FXMA108, Package_DFN_QFN:WQFN-20-1EP_2.5x4.5mm_P0.5mm_EP1x2.9mm, symbol Logic_LevelTranslator:FXMA108
- added U9: PCAL6416AHF, Package_DFN_QFN:HVQFN-24-1EP_4x4mm_P0.5mm_EP2.1x2.1mm, symbol Interface_Expansion:PCAL6416AHF
- J1: footprint Connector_BarrelJack:BarrelJack_CUI_PJ-036AH-SMT_Horizontal -> CUI_PJ-036AH-SMT-TR
- J3: renamed from J11; value Conn_01x08_Pin -> Conn_01x10_Pin; footprint Connector_PinHeader_2.54mm:PinHeader_2x08_P2.54mm_Vertical -> Connector_PinHeader_2.54mm:PinHeader_1x10_P2.54mm_Vertical; symbol Connector:Conn_01x08_Pin -> Connector:Conn_01x10_Pin
- R23, R25, R32, R34: value 1K -> 10K
- R24, R26, R33: value 1K -> 20K
- renumbered C11 to C1, C5 to C10, C6 to C11, C17 to C12, C18 to C13, C15 to C14, C9 to C15, C4 to C16, C16 to C17, C10 to C18, C1 to C2, C2 to C3, C12 to C4, C13 to C5, C14 to C6, C3 to C7, C7 to C8, C8 to C9, D3 to D1, D4 to D2, J8 to J10, J13 to J11, J9 to J12, J10 to J13, J3 to J4, J4 to J6, J6 to J7, J12 to J8, J7 to J9, R9 to R1, R3 to R11, R4 to R12, R11 to R19, R7 to R2, R6 to R20, R2 to R3, R12 to R4, R13 to R5, R1 to R6, SW3 to SW1, SW1 to SW2, SW2 to SW3, TP2 to TP1, TP3 to TP2, U5 to U1, U3 to U2, U6 to U3, U7 to U4, U2 to U6, U4 to U7
Connections:
- net +3.3V: now also J3.9 (Pin_9), C19.1, C21.1, C22.1, C24.1, C25.1, MT1.5 (VDDIO), MT1.8 (VDD), R36.1, R37.1, R38.1, R44.1, R45.1, R46.1, R49.1, U5.2 (3V3), U8.1 (VCCA), U9.23 (V_{DD(I2C-bus)}); no longer J10.5, J11.5, J12.5, J13.5, J3.5 (Pin_5), J3.6 (Pin_6), J4.5, J5.5, J6.5, J7.5, J8.5, J9.5
- net +5V: now also J10.4, J11.4, J12.4, J13.4, J4.4, J5.4, J6.4, J7.4, J8.4, J9.4, C20.2, C23.2, U8.20 (VCCB), U9.21 (V_{DD(P)}); no longer J3.7 (Pin_7)
- net +6V: now also J4.3, J5.3, J6.3, J7.3; no longer J4.4, J5.4, J6.4, J7.4
- net D+: now also U5.14 (GPIO20/U1CTS/ADC2_CH9/CLK_OUT1/USB_D+)
- net D-: now also U5.13 (GPIO19/U1RTS/ADC2_CH8/CLK_OUT2/USB_D-)
- net GND: now also J10.5, J11.5, J12.5, J13.5, J3.10 (Pin_10), J4.5, J5.5, J6.5, J7.5, J8.5, J9.5, R24.2, R26.2, R31.2, R33.2, C19.2, C20.1, C21.2, C22.2, C23.1, C24.2, C25.2, MT1.6 (GND), R35.2, R39.2, R43.2, R47.2, R52.2, U5.1 (GND), U5.40 (GND), U5.41 (GND), U8.10 (GND), U9.25 (EP), U9.9 (V_{SS}); no longer J10.6, J11.6, J12.6, J13.6, J3.8 (Pin_8), J4.6, J5.6, J6.6, J7.6, J8.6, J9.6
- net GPIO1: now also R25.2, R26.1, U5.39 (GPIO1/TOUCH1/ADC1_CH0)
- net GPIO10: now also J3.4 (Pin_4), U5.18 (GPIO10/TOUCH10/ADC1_CH9/FSPICS0/FSPIIO4/SUBSPICS0); no longer R28.2
- net GPIO11: now also J3.5 (Pin_5), U5.19 (GPIO11/TOUCH11/ADC2_CH0/FSPID/FSPIIO5/SUBSPID); no longer R29.2
- net GPIO12: now also J3.6 (Pin_6), U5.20 (GPIO12/TOUCH12/ADC2_CH1/FSPICLK/FSPIIO6/SUBSPICLK); no longer R30.2
- net GPIO13: now also J3.7 (Pin_7), U5.21 (GPIO13/TOUCH13/ADC2_CH2/FSPIQ/FSPIIO7/SUBSPIQ); no longer R31.1
- net GPIO14: now also J3.8 (Pin_8), U5.22 (GPIO14/TOUCH14/ADC2_CH3/FSPIWP/FSPIDQS/SUBSPIWP); no longer R32.1
- net GPIO15: now also R45.2, U5.8 (GPIO15/U0RTS/ADC2_CH4/XTAL_32K_P), U9.19 (SCL); no longer R33.1
- net GPIO16: now also R44.2, U5.9 (GPIO16/U0CTS/ADC2_CH5/XTAL_32K_N), U9.20 (SDA); no longer R34.1
- net GPIO17: now also MT1.13 (AP_SCL/AP_SCLK), R37.2, U5.10 (GPIO17/U1TXD/ADC2_CH6)
- net GPIO18: now also MT1.14 (AP_SDA/AP_SDIO/AP_SDI), R36.2, U5.11 (GPIO18/U1RXD/ADC2_CH7/CLK_OUT3); no longer R8.2
- net GPIO2: now also R32.2, R33.1, U5.38 (GPIO2/TOUCH2/ADC1_CH1)
- net GPIO3: now also R42.2, R43.1, U5.15 (GPIO3/TOUCH3/ADC1_CH2); no longer R21.2
- net GPIO35: now also U5.28 (SPIIO6/GPIO35/FSPID/SUBSPID), U8.2 (A0); no longer R14.2
- net GPIO36: now also U5.29 (SPIIO7/GPIO36/FSPICLK/SUBSPICLK), U8.3 (A1); no longer R15.2
- net GPIO37: now also U5.30 (SPIDQS/GPIO37/FSPIQ/SUBSPIQ), U8.4 (A2); no longer U3.6 (IN1/PH)
- net GPIO38: now also U5.31 (GPIO38/FSPIWP/SUBSPIWP), U8.5 (A3); no longer U3.5 (IN2/EN)
- net GPIO39: now also U5.32 (MTCK/GPIO39/CLK_OUT3/SUBSPICS1), U8.6 (A4); no longer U6.6 (IN1/PH)
- net GPIO4: now also R51.2, R52.1, U5.4 (GPIO4/TOUCH4/ADC1_CH3); no longer R22.2
- net GPIO40: now also U5.33 (MTDO/GPIO40/CLK_OUT2), U8.7 (A5); no longer U6.5 (IN2/EN)
- net GPIO41: now also U3.6 (IN1/PH), U5.34 (MTDI/GPIO41/CLK_OUT1), U8.8 (A6); no longer U4.6 (IN1/PH)
- net GPIO42: now also U3.5 (IN2/EN), U5.35 (MTMS/GPIO42), U8.9 (A7); no longer U4.5 (IN2/EN)
- net GPIO43: now also U6.6 (IN1/PH), U5.37 (U0TXD/GPIO43/CLK_OUT1); no longer U7.6 (IN1/PH)
- net GPIO44: now also U6.5 (IN2/EN), U5.36 (U0RXD/GPIO44/CLK_OUT2); no longer U7.5 (IN2/EN)
- net GPIO45: now also U4.6 (IN1/PH), U5.26 (GPIO45); no longer R16.2
- net GPIO5: now also R24.1, U5.5 (GPIO5/TOUCH5/ADC1_CH4)
- net GPIO6: now also R34.2, R35.1, U5.6 (GPIO6/TOUCH6/ADC1_CH5); no longer R24.2
- net GPIO7: now also J3.1 (Pin_1), U5.7 (GPIO7/TOUCH7/ADC1_CH6); no longer R25.2
- net GPIO8: now also J3.2 (Pin_2), U5.12 (GPIO8/TOUCH8/ADC1_CH7/SUBSPICS1); no longer R26.2
- net GPIO9: now also J3.3 (Pin_3), U5.17 (GPIO9/TOUCH9/ADC1_CH8/FSPIHD/SUBSPIHD); no longer R27.2
- net at R14.1: now also J6.7; no longer J5.8
- net at J11.8: now also R34.1; no longer R30.1
- net at R15.1: now also J7.6; no longer J7.7
- net at R16.1: now also J7.7; no longer J7.8
- net at C16.1, SW3.1: now also U5.27 (GPIO0/BOOT)
- net at R17.1: now also J8.6; no longer J6.7
- net at R18.1: now also J8.7; no longer J6.8
- net at C7.2, R6.2, SW2.2: now also U5.3 (EN)
- net at J9.7: now also R22.1
- net at J9.8: now also R25.1
- net at R27.1: now also J11.6; no longer J8.7
- net at J12.7: now also R41.1; no longer R23.1
- net at R21.1: now also J9.6; no longer J10.7
- net at J10.8: now also R32.1; no longer R22.1
- net at J13.8: now also R51.1; no longer R26.1
- net at J13.7: now also R50.1; no longer R25.1
- net at J12.8: now also R42.1; no longer R24.1
- net at R28.1: now also J10.6; no longer J8.8
- net at R8.1: now also J4.7; no longer J4.8
- net GPIO21 renamed EXP10
- net EXP10: now also U9.10 (P1_0)
- net GPIO33 renamed EXP11
- net EXP11: now also U9.11 (P1_1)
- net GPIO34 renamed ENC3B
- net ENC3B: now also U9.6 (P0_5)
- new net: J4.6, R7.1
- new net: R47.1, U9.18 (ADDR)
- new net: R49.2, U9.22 (~{INT})
- new net: R46.2, U9.24 (~{RESET})
- new net: J12.6, R40.1
- new net: MT1.12 (AP_CS), R38.2
- new net: J10.7, R30.1
- new net: J6.6, R13.1
- new net: J8.8, R23.1
- new net: J5.6, R9.1
- new net: J13.6, R48.1
- new net: MT1.1 (AP_SDO/AP_AD0), R39.1
- new net: R31.1, U8.11 (~{OE})
- new net B0: R21.2, U8.19 (B0)
- new net B1: R22.2, U8.18 (B1)
- new net B2: R28.2, U8.17 (B2)
- new net B3: R30.2, U8.16 (B3)
- new net B4: R40.2, U8.15 (B4)
- new net B5: R41.2, U8.14 (B5)
- new net B6: R48.2, U8.13 (B6)
- new net B7: R50.2, U8.12 (B7)
- new net ENC1A: R7.2, U9.1 (P0_0)
- new net ENC1B: R8.2, U9.2 (P0_1)
- new net ENC2A: R13.2, U9.3 (P0_2)
- new net ENC2B: R14.2, U9.4 (P0_3)
- new net ENC3A: R9.2, U9.5 (P0_4)
- new net ENC4A: R15.2, U9.7 (P0_6)
- new net ENC4B: R16.2, U9.8 (P0_7)
- new net EXP12: R27.2, U9.12 (P1_2)
- new net EXP13: R29.2, U9.13 (P1_3)
- new net GPIO46: U4.5 (IN2/EN), U5.16 (GPIO46)
- new net GPIO47: U5.24 (GPIO47/SPICLK_P/SUBSPICLK_P_DIFF), U7.6 (IN1/PH)
- new net GPIO48: U5.25 (GPIO48/SPICLK_N/SUBSPICLK_N_DIFF), U7.5 (IN2/EN)
- no-connect marks 32 -> 37
Other:
- moved on the sheet: J10, J11, J12, J13, J8, J9
